Commit message: Hasta la polla

File: Fisica-II/robot/robot.urdf (robot description, URDF)
Before this commit: robot libro, 8 links, 7 joints
Links:
- link link0: geometry visual cylinder length=0.1 radius=0.1
- link link1: geometry visual box size=0.1 0.1 0.2
- link link2: geometry visual box size=0.1 0.1 0.5
- link link3: geometry visual box size=0.1 0.1 0.5
- link link5: geometry visual cylinder length=0.2 radius=0.05
- link link7: geometry visual box size=0.1 0.1 0.2
Joints:
- joint joint1: limit lower=-1.57 upper=1.57 effort=100.0 velocity=1.0 -> lower=-3.14 upper=3.14 effort=100.0 velocity=1.0; origin xyz=0 0 0.5 rpy=0 0 0 -> xyz=0 0 0 rpy=0 0 0
- joint joint2: origin xyz=0 0 1 rpy=0 0 0 -> xyz=0 0 0.2 rpy=0 0 0
- joint joint3: axis 0 0 0 -> 1 0 0; origin xyz=0 0 0 rpy=0 0 0 -> xyz=0 0 0.5 rpy=0 0 0; type prismatic -> revolute
- joint joint4: axis 1 0 0 -> 0 1 0; origin xyz=0 1 1 rpy=0 0 0 -> xyz=0 0.5 0 rpy=0 0 0; type revolute -> prismatic
- joint joint5: limit lower=-1.57 upper=1.57 effort=100.0 velocity=1.0 -> lower=0 upper=0.2 effort=100.0 velocity=1.0; origin xyz=0 1.5 1 rpy=0 0 0 -> xyz=0 0.3 0 rpy=0 0 0; type revolute -> prismatic
- joint joint6: axis 0 0 0 -> 0 1 0; origin xyz=0 0 0 rpy=0 0 0 -> xyz=0 0.2 0 rpy=0 0 0; type prismatic -> revolute
- joint joint7: origin xyz=0 2.5 1 rpy=0 0 0 -> xyz=0 0.5 0 rpy=0 0 0
